File: kicad/cmd_module_booster/cmd_module_booster.kicad_pcb (KiCad board)
At the start: 2 copper layers, 15 parts, among them J1 Rails, J2 Power, J3 RPi Connect, U1 LMD18200

Commit message: Add step model of command booster
Other:
- board outline added: 63.5 x 81.3 mm
